File: USB_DAC1.sch (KiCad schematic (older format))
At the start: 57 parts

Commit message: ボードを追加
Parts:
- removed J?: USB_A, symbol USB_A
- removed R? (x4): 1k, symbol R
- removed RV? (x2): POT, symbol POT
- removed U? (x2): 7805, symbol 7805
- added C10, C11, C16, C25, C26, C28, C29, C31, C32, C33, C35, C37: 1u, Capacitors_SMD:C_0805_HandSoldering, symbol C_Small
- added C18, C19, C23, C3: 100u, Discret:C1V8, symbol CP_Small
- added C27, C34: 1500u, Discret:C2V8, symbol CP_Small
- added J1: USB_OTG, Connectors_Molex:USB_Micro-B_Molex_47346-0001, symbol USB_OTG
- added L10, L3, L4, L7, L8, L9: 4.7u, Inductors:INDUCTOR_V, symbol L
- added R1: 1M, Discret:R3, symbol R_Small
- added R10, R11, R12, R13, R14, R16, R20, R22, R3, R4: 1, Discret:R3, symbol R
- added R26, R27: 1k, Discret:R3, symbol R
- added RV1: 10k, Potentiometers:Potentiometer_Alps_RK097_Double_Vertical, symbol POT_Dual
- added U2, U3: MC78M05CDT, TO_SOT_Packages_SMD:TO-252-2Lead, symbol MC78M05CDT
- C1, C2: renamed from C?; footprint (none) -> Pin_Headers:Pin_Header_Straight_1x02_Pitch2.54mm
- C12, C14, C15: renamed from C?; value C_Small -> 1u; footprint (none) -> Capacitors_SMD:C_0805_HandSoldering
- C13, C22, C24: renamed from C?; value CP_Small -> 100u; footprint (none) -> Discret:C1V8
- C17, C8: renamed from C?; value CP_Small -> 1500u; footprint (none) -> Discret:C2V8
- C20, C21: renamed from C?; value C_Small -> 0.1u; footprint (none) -> Capacitors_SMD:C_0805_HandSoldering
- C30, C36: renamed from C?; value C_Small -> 2200p; footprint (none) -> Pin_Headers:Pin_Header_Straight_1x02_Pitch2.54mm
- C4, C5, C7, C9: renamed from C?; value 10u -> 1u; footprint (none) -> Capacitors_SMD:C_0805_HandSoldering
- C6: renamed from C?; value CP_Small -> 1000u; footprint (none) -> Discret:C2V8
- D1: renamed from D?; footprint (none) -> LEDs:LED_0603
- J2: renamed from J?; footprint (none) -> mylib:35_TRS
- J3: renamed from J?; footprint (none) -> mylib:TRRS_1
- L1, L2, L5, L6: renamed from L?; value L -> 4.7u; footprint (none) -> Inductors:INDUCTOR_V
- R15, R17, R18, R21, R23, R24: renamed from R?; value R -> 1k; footprint (none) -> Discret:R3
- R19, R25: renamed from R?; value R -> 2k; footprint (none) -> Discret:R3
- R2: renamed from R?; value R_Small -> 1k; footprint (none) -> Discret:R3
- R5: renamed from R?; value R_Small -> 10k; footprint (none) -> Discret:R3
- R6, R9: renamed from R?; value R -> 22; footprint (none) -> Discret:R3
- R7: renamed from R?; footprint (none) -> Discret:R3
- R8: renamed from R?; value R -> 1; footprint (none) -> Discret:R3
- U1: renamed from U?; footprint (none) -> Housings_SSOP:SSOP-28_5.3x10.2mm_Pitch0.65mm
- U4, U5, U6: renamed from U?; footprint (none) -> Housings_DIP:DIP-8_W7.62mm
- Y1: renamed from Y?; footprint (none) -> Crystals:Crystal_HC18-U_Vertical
Connections:
- net GNDA: now also C18.2, C19.2, C23.2, C3.2, J1.5 (GND), L10.1, L4.2, L8.1, U2.2 (GND), U3.2 (GND); no longer C17.2, L2.2, U4.4 (V-), U4.4 (V-), U5.4 (V-), U5.4 (V-), U6.4 (V-), U6.4 (V-)
- net L_COLD: now also U6.7; no longer U6.1
- net R_COLD: now also U5.7; no longer U5.1
- net VBUS: now also C3.1, J1.1 (VBUS), R3.2; no longer U1.10 (VBUS)
- net VDD: now also U1.10 (VBUS), U2.3 (OUT)
- net VDDA: now also C22.1, C24.1, L3.2, L7.1, L9.1, R11.2, R12.1, U3.3 (OUT); no longer C20.1, C21.1, C8.1, L5.1, L6.2, U4.8 (V+), U4.8 (V+), U5.8 (V+), U5.8 (V+), U6.8 (V+), U6.8 (V+)
- net at C1.1, U1.1 (XTO), Y1.1: now also R1.2
- net at L5.2, U1.13 (VCCL): now also C20.1; no longer C22.1
- net at U1.14 (VOUTL): now also R27.2; no longer R24.2
- net at U1.15 (VOUTR): now also R26.1; no longer R18.2
- net at L6.1, U1.16 (VCCR): now also C21.1; no longer C24.1
- net at C12.1, R7.2, U1.18 (VCOM): now also C18.1
- net at C2.1, U1.28 (XTI), Y1.2: now also R1.1
- net at R6.2: now also J1.2 (D-)
- net at R9.2: now also J1.3 (D+)
- net at C5.2, L1.2: now also U2.1 (IN)
- net at C9.1, L2.1: now also U3.1 (IN)
- net at R8.2, U4.1, U4.2 (-): no longer U4.3 (+)
- net at C13.1, C15.1, R7.1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: now also U4.5 (+)
- net at C36.2, R24.1, R25.2: now also U6.6 (-); no longer U6.2 (-)
- net GND: now reaches U6.3 (+)
- net GND: now also C17.1, C8.2, J2.3, R8.1, U5.3 (+), U5.5 (+), U6.5 (+), C10.2, C16.1, C25.2, C29.2, C31.2, C35.1, R13.2, RV1.1, RV1.2, RV1.4, RV1.5; no longer U6.3 (+)
- net at C30.2, R18.1, R19.2: now also U5.6 (-); no longer U5.2 (-)
- new net: C19.1, L6.2, R12.2
- new net: C23.1, L5.1, R11.1
- new net: C16.2, C17.2, C37.2, R10.2, U4.4 (V-)
- new net: C10.1, C37.1, C8.1, R4.2, U4.8 (V+)
- new net: C33.1, C34.2, C35.2, R22.2, U6.4 (V-)
- new net: C31.1, C33.2, C34.1, R20.2, U6.8 (V+)
- new net: C26.1, C27.2, C29.1, R16.2, U5.4 (V-)
- new net: C25.1, C26.2, C27.1, R14.2, U5.8 (V+)
- new net: R24.2, R27.1, RV1.6
- new net: R18.2, R26.2, RV1.3
- new net: R13.1, U4.6 (-), U4.7
- new net: L2.2, R3.1
- new net: C28.1, L8.2, R16.1
- new net: C28.2, L7.2, R14.1
- new net: C32.2, L9.2, R20.1
- new net: C11.1, L3.1, R4.1
- new net: C32.1, L10.2, R22.1
- new net: C11.2, L4.1, R10.1
- no-connect marks 6 -> 8
Other:
- moved on the sheet: C20, C21, C22, C24
